File: Electronics/main_PCB_v1/main_PCB_v1.kicad_sch (KiCad schematic)
At the start: 1 part

Commit message: PCB Finished
Changed lines of the file:
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@@
+    (stroke (width 0) (type default))
+  )
+  (wire (pts (xy 149.86 160.02) (xy 149.86 162.56))
+    (stroke (width 0) (type default))
+  )
+  (wire (pts (xy 149.86 162.56) (xy 160.02 162.56))
+    (stroke (width 0) (type default))
+  )
+  (wire (pts (xy 111.76 76.2) (xy 144.78 76.2))
     (stroke (width 0) (type default))
   )
@@
     (stroke (width 0) (type default))
   )
+  (wire (pts (xy 111.76 73.66) (xy 144.78 73.66))
+    (stroke (width 0) (type default))
+  )
   (bus (pts (xy 185.42 73.66) (xy 205.74 73.66))
+    (stroke (width 0) (type default))
+  )
+  (wire (pts (xy 160.02 160.02) (xy 160.02 162.56))
     (stroke (width 0) (type default))
   )
@@
     )
   )
+  (symbol (lib_id "power:+3V3") (at 149.86 160.02 0) (unit 1)
+    (in_bom yes) (on_board yes) (dnp no) (fields_autoplaced)
+    (property "Reference" "#PWR0103" (at 149.86 163.83 0)
+      (effects (font (size 1.27 1.27)) hide)
+    )
+    (property "Value" "+3V3" (at 149.86 154.94 0)
+      (effects (font (size 1.27 1.27)))
+    )
+    (property "Footprint" "" (at 149.86 160.02 0)
+      (effects (font (size 1.27 1.27)) hide)
+    )
+    (property "Datasheet" "" (at 149.86 160.02 0)
+      (effects (font (size 1.27 1.27)) hide)
+    )
+    (pin "1")
+    (instances
+      (project "main_PCB_v1"
+        (path "/73132c36-f9bc-41a1-bd49-e7f0b5a0c66e"
+          (reference "#PWR0103") (unit 1)
+        )
+      )
+    )
+  )
   (symbol (lib_id "power:GND") (at 127 167.64 0) (unit 1)
     (in_bom yes) (on_board yes) (dnp no) (fields_autoplaced)
@@
         )
       )
+    )
+  )
+  (symbol (lib_id "power:+3.3V") (at 160.02 160.02 0) (unit 1)
+    (in_bom yes) (on_board yes) (dnp no) (fields_autoplaced)
+    (property "Reference" "#PWR0104" (at 160.02 163.83 0)
+      (effects (font (size 1.27 1.27)) hide)
+    )
+    (property "Value" "+3.3V" (at 160.02 154.94 0)
+      (effects (font (size 1.27 1.27)))
+    )
+    (property "Footprint" "" (at 160.02 160.02 0)
+      (effects (font (size 1.27 1.27)) hide)
+    )
+    (property "Datasheet" "" (at 160.02 160.02 0)
+      (effects (font (size 1.27 1.27)) hide)
+    )
+    (pin "1")
+    (instances
+      (project "main_PCB_v1"
+        (path "/73132c36-f9bc-41a1-bd49-e7f0b5a0c66e"
+          (reference "#PWR0104") (unit 1)
+        )
+      )
