File: Electronics/main_PCB_v1/microcontroller.kicad_sch (KiCad schematic)
At the start: 83 parts, among them IC302 TJA1057GT/3, IC303 TJA1057GT/3, J203 TYPE-C-31-M-12, J204 Conn_02x04_Odd_Even, J205 Conn_ST_STDC14, J207 Conn_01x04, J208 SM02B-GHS-TB_LF__SN_, J209 SM02B-GHS-TB_LF__SN_, J210 SM02B-GHS-TB_LF__SN_, J211 SM02B-GHS-TB_LF__SN_, J212 SM02B-GHS-TB_LF__SN_, J302 MEM2075-00-140-01-A, U201 STM32H723ZGT6, U202 USBLC6-4SC6, U203 USBLC6-4SC6, U204 BMI270, U211 M24C08-FMH6TG, U404 LIS3MDL, X201 25MHz_Clock, X202 32.768kHz_Clock

Commit message: PCB Finished
Connections:
- net +3V3: now also J204.8 (Pin_8); no longer J204.4 (Pin_4)
- net +5V: now also J204.4 (Pin_4); no longer J204.8 (Pin_8)
- net BTN1: now also U201.34 (PA0)
- net BTN2: now also U201.44 (PC4)
- net LEDB: now also U201.134 (PB4)
- net LEDG: now also U201.132 (PG15)
- net LEDR: now also U201.129 (PG14)
- net NRF24_IRQ: now also U201.80 (PD11)
- net TRIG1: now also U201.41 (PA5)
- net TRIG2: now also U201.35 (PA1)
- net GPIO3: now reaches U201.18 (PF6)
- net GPIO3: now also J204.5 (Pin_5)
- net GPIO4: now reaches U201.19 (PF7)
- net GPIO4: now also J204.6 (Pin_6)
- net GPIO2: now reaches U201.20 (PF8)
- net GPIO2: now also J204.2 (Pin_2)
- net GPIO1: now reaches U201.21 (PF9)
- net GPIO1: now also J204.1 (Pin_1)
- no-connect marks 21 -> 75
Other:
- moved on the sheet: U201A
