File: Electronics/main_PCB_v2/power.kicad_sch (KiCad schematic)
At the start: 60 parts, among them J301 Conn_01x02, J302 Conn_01x02, J305 Conn_01x02, J306 Conn_01x02, J307 Conn_01x02, J308 Conn_01x02, J309 Conn_01x02, J310 Conn_01x02, Q302 DMP3028LFDE, T301 NVMFS4C05NT1G, T302 NVMFS4C05NT1G, U301 LMR43620MB5RPER, U302 LMR43620MB5RPER, U303 LMR43620MB5RPER, U304 TVS2700DRV

Commit message: New board requirements
Parts:
- added C325: 100u, Capacitor_SMD:CP_Elec_6.3x7.7, symbol Device:C_Polarized_Small
Changed lines of the file:
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@@
     (stroke (width 0) (type default))
   )
-  (text_box "Input capacitors must be rated for >24V"
+  (text_box "Input capacitors must be rated for >25V"
     (at 165.1 68.58 0) (size 20.32 7.62)
     (stroke (width 0) (type default))
@@
         )
       )
+    )
+  )
+  (symbol (lib_id "Device:C_Polarized_Small") (at 124.46 124.46 0) (unit 1)
+    (in_bom yes) (on_board yes) (dnp no) (fields_autoplaced)
+    (property "Reference" "C325" (at 127 122.6439 0)
+      (effects (font (size 1.27 1.27)) (justify left))
+    )
+    (property "Value" "100u" (at 127 125.1839 0)
+      (effects (font (size 1.27 1.27)) (justify left))
+    )
+    (property "Footprint" "Capacitor_SMD:CP_Elec_6.3x7.7" (at 124.46 124.46 0)
+      (effects (font (size 1.27 1.27)) hide)
+    )
+    (property "Datasheet" "~" (at 124.46 124.46 0)
+      (effects (font (size 1.27 1.27)) hide)
+    )
+    (pin "2")
+    (pin "1")
+    (instances
+      (project "main_PCB_v2"
+        (path "/73132c36-f9bc-41a1-bd49-e7f0b5a0c66e/0967cea5-ca64-435c-884b-84cde77959f6"
+          (reference "C325") (unit 1)
+        )
+      )
