File: Electronics/stacked_board_power_v1/main_PCB_v2.kicad_pcb (KiCad board)
At the start: 4 copper layers, 100 x 95.5 mm, 254 parts, among them IC202 TJA1057GT/3, IC203 TJA1057GT/3, J101 Conn_01x02, J102 Conn_01x02, J104 Conn_01x02, J105 Conn_01x02, J106 Conn_01x02, J108 Conn_01x02, J109 Conn_02x20_Odd_Even, J201 MEM2075-00-140-01-A, J203 TYPE-C-31-M-12, J204 Conn_02x04_Odd_Even, J205 Conn_ST_STDC14, J207 Conn_01x04, J208 SM02B-GHS-TB_LF__SN_, J209 SM02B-GHS-TB_LF__SN_, J210 SM02B-GHS-TB_LF__SN_, J211 SM02B-GHS-TB_LF__SN_, J212 SM02B-GHS-TB_LF__SN_, J301 Conn_01x02, J302 Conn_01x02, J305 Conn_01x02, J306 Conn_01x02, J307 Conn_01x02, J308 Conn_01x02, J309 Conn_01x02, J310 Conn_01x02, J401 Conn_Coaxial, K101 G2RL-1-E, Q302 DMP3028LFDE, T301 NVMFS4C05NT1G, T302 NVMFS4C05NT1G, U101 TVS2700DRV, U102 TPS16416DRCR, U103 LMR43620MB5RPER, U104 LMR43620MB5RPER, U105 LMR43620MB5RPER, U106 TPS25961DRVR, U107 TPS25961DRVR, U201 STM32H723ZGT6, U202 USBLC6-4SC6, U203 USBLC6-4SC6, U204 BMI270, U206 LIS3MDL, U211 M24C08-FMH6TG, U301 LMR43620MB5RPER, U302 LMR43620MB5RPER, U303 LMR43620MB5RPER, U401 NRF24L01, U402 RFX2401C, X201 25MHz_Clock, X202 32.768kHz_Clock, Y402 16M

Commit message: Power board done
Parts:
- removed AE401: Antenna, SSL Footprints:Texas_SWRA117D_2.4GHz_Right
- removed C201, C202, C205, C206, C207, C208, C209, C210, C212, C213, C214, C215, C216, C217, C218, C223, C224, C225, C226, C227, C228, C229, C231, C232, C233, C235, C237, C238, C302, C304, C312, C318, C321, C322: 100n, Capacitor_SMD:C_0402_1005Metric
- removed C203, C204, C220, C221, C401, C408: 10n, Capacitor_SMD:C_0402_1005Metric
- removed C211, C219, C222: 10u, Capacitor_SMD:C_0402_1005Metric
- removed C230, C234, C236, C303, C311, C317, C409: 1u, Capacitor_SMD:C_0402_1005Metric
- removed C301, C313, C316: 2u2, Capacitor_SMD:C_0603_1608Metric
- removed C305, C306, C314, C315, C319, C320: 22u, Capacitor_SMD:C_0603_1608Metric
- removed C307, C308, C309: 100p, Capacitor_SMD:C_0402_1005Metric
- removed C310, C323, C324, C406: 1n, Capacitor_SMD:C_0402_1005Metric
- removed C402, C414, C415, C416, C417: 1p5, Capacitor_SMD:C_0402_1005Metric
- removed C403: 1p, Capacitor_SMD:C_0402_1005Metric
- removed C404: 2n2, Capacitor_SMD:C_0402_1005Metric
- removed C405: 4p7, Capacitor_SMD:C_0402_1005Metric
- removed C407: 33n, Capacitor_SMD:C_0402_1005Metric
- removed C410, C411: 22p, Capacitor_SMD:C_0402_1005Metric
- removed C412: 220p, Capacitor_SMD:C_0402_1005Metric
- removed C413: 0p3, Capacitor_SMD:C_0402_1005Metric
- removed D201: SS0540_R1_00001, Diode_SMD:D_SOD-123
- removed D202: Red, LED_SMD:LED_0603_1608Metric
- removed D203, D301, D302, D304: Green, LED_SMD:LED_0603_1608Metric
- removed D204: Blue, LED_SMD:LED_0603_1608Metric
- removed D303: ZMM10V, Diode_SMD:D_MiniMELF
- removed FB201: 120R@100MHz, Resistor_SMD:R_0402_1005Metric
- removed FL201: EMIF06-MSD02N16, SSL Footprints:EMIF06MSD02N16
- removed the G*** at (139.6, 91.2)
- removed the G*** at (137.8, 86.6)
- removed IC202, IC203: TJA1057GT/3, SSL Footprints:SOIC127P600X175-8N
- removed J201: MEM2075-00-140-01-A, SSL Footprints:MEM20750014001A
- removed J203: TYPE-C-31-M-12, SSL Footprints:HRO_TYPE-C-31-M-12
- removed J204: Conn_02x04_Odd_Even, Connector_PinHeader_2.54mm:PinHeader_2x04_P2.54mm_Vertical
- removed J205: Conn_ST_STDC14, Connector_PinHeader_1.27mm:PinHeader_2x07_P1.27mm_Vertical
- removed J207: Conn_01x04, Connector_PinHeader_2.54mm:PinHeader_1x04_P2.54mm_Vertical
- removed J208, J209, J210, J211, J212: SM02B-GHS-TB_LF__SN_, SSL Footprints:SM02BGHSTBLFSN
- removed J301: Conn_01x02, Connector_AMASS:AMASS_XT60-M_1x02_P7.20mm_Vertical
- removed J302, J305, J306, J307, J308, J309, J310: Conn_01x02, Connector_AMASS:AMASS_XT30U-F_1x02_P5.0mm_Vertical
- removed J401: Conn_Coaxial, SSL Footprints:SMA_Amphenol_901-143_Horizontal
- removed L301, L303, L305: 4u7, Inductor_SMD:L_Chilisin_BMRA00040420
- removed L401: 3n9, Inductor_SMD:L_0402_1005Metric
- removed L402, L405: 2n4, Inductor_SMD:L_0402_1005Metric
- removed L403: 8n2, Inductor_SMD:L_0402_1005Metric
- removed L404: 2n7, Inductor_SMD:L_0402_1005Metric
- removed OL101: Main_board_outline_v2, SSL Footprints:main_board_outline_v2
- removed Q302: DMP3028LFDE, SSL Footprints:DMP2066UFDE7
- removed R108, R205, R206, R207, R210, R304, R314, R315: 10k, Resistor_SMD:R_0402_1005Metric
- removed R120: 6k8, Resistor_SMD:R_0402_1005Metric
- removed R121, R124, R308: 49k9, Resistor_SMD:R_0402_1005Metric
- removed R122, R123: k, Resistor_SMD:R_0402_1005Metric
- removed R201, R202: 5k1, Resistor_SMD:R_0402_1005Metric
- removed R203, R204, R214, R215, R305: 4k7, Resistor_SMD:R_0402_1005Metric
- removed R208, R209: 120R, Resistor_SMD:R_0402_1005Metric
- removed R211, R212, R213: 2k7, Resistor_SMD:R_0402_1005Metric
- removed R301: 120k, Resistor_SMD:R_0402_1005Metric
- removed R302: 11k, Resistor_SMD:R_0402_1005Metric
- removed R303, R401, R405, R406, R407: 22k, Resistor_SMD:R_0402_1005Metric
- removed R307: 2k2, Resistor_SMD:R_0402_1005Metric
- removed R309: 12k4, Resistor_SMD:R_0402_1005Metric
- removed R310: 33k, Resistor_SMD:R_0402_1005Metric
- removed R311: 14k3, Resistor_SMD:R_0402_1005Metric
- removed R312, R313: 10R, Resistor_SMD:R_0402_1005Metric
- removed R402: 1M, Resistor_SMD:R_0402_1005Metric
- removed R403, R404: 1k, Resistor_SMD:R_0402_1005Metric
- removed S201, S202, S203, S204: TS20-42-25-WT-160-SMT-TR, SSL Footprints:TS204225WT160SMTTRMSL
- removed S401: SKY13453-385LF, SSL Footprints:SKY13453385LF
- removed SH401: SMS-202F, SSL Footprints:SMS202F
- removed T301, T302: NVMFS4C05NT1G, SSL Footprints:TRANS_NVMFS5834NLWFT1G
- removed U106, U107: TPS25961DRVR, SSL Footprints:SON65P200X200X80-7N
- removed U201: STM32H723ZGT6, SSL Footprints:QFP50P2200X2200X160-144N
- removed U202, U203: USBLC6-4SC6, Package_TO_SOT_SMD:SOT-23-6
- removed U204: BMI270, SSL Footprints:BMI270_BOS
- removed U206: LIS3MDL, Package_LGA:LGA-12_2x2mm_P0.5mm
- removed U211: M24C08-FMH6TG, SSL Footprints:M24C08FMH6TG
- removed U301, U302, U303: LMR43620MB5RPER, SSL Footprints:LMR43620MB5RPER_TEX
- removed U401: NRF24L01, Package_DFN_QFN:QFN-20-1EP_4x4mm_P0.5mm_EP2.5x2.5mm
- removed U402: RFX2401C, SSL Footprints:QFN50P300X300X60-17N-D
- removed X201: 25MHz_Clock, Oscillator:Oscillator_SMD_Abracon_ASE-4Pin_3.2x2.5mm
- removed X202: 32.768kHz_Clock, Oscillator:Oscillator_SMD_Abracon_ASE-4Pin_3.2x2.5mm
- removed Y402: 16M, Oscillator:Oscillator_SMD_Abracon_ASE-4Pin_3.2x2.5mm
- added C130: 100n, Capacitor_SMD:C_0402_1005Metric, F.Cu at (160.0, 121.8)
- added C131: 100n, Capacitor_SMD:C_0402_1005Metric, F.Cu at (157.2, 85.5)
- added C132: 330n, Capacitor_SMD:C_0402_1005Metric, F.Cu at (156.2, 85.5)
- added C133: 330n, Capacitor_SMD:C_0402_1005Metric, F.Cu at (167.2, 85.5)
- added C134: 100n, Capacitor_SMD:C_0402_1005Metric, F.Cu at (168.2, 85.5)
- added D102: SS0540_R1_00001, Diode_SMD:D_SOD-123, F.Cu at (128.8, 52.0)
- added D106: RFN1LAM6STR, Diode_SMD:D_SOD-128, F.Cu at (143.5, 90.8)
- added G***: LOGO, SSL Footprints:ICRS_30mm, B.Cu at (155.0, 69.5)
- added J103: Conn_01x02, Connector_AMASS:AMASS_XT30U-F_1x02_P5.0mm_Vertical, F.Cu at (130.8, 91.4)
- added J107: Conn_01x02, Connector_AMASS:AMASS_XT30U-F_1x02_P5.0mm_Vertical, F.Cu at (138.3, 104.4)
- added J110: Conn_01x02, Connector_AMASS:AMASS_XT30U-F_1x02_P5.0mm_Vertical, F.Cu at (134.5, 97.9)
- added J111: Conn_02x03_Counter_Clockwise, Connector_IDC:IDC-Header_2x03_P2.54mm_Vertical, F.Cu at (151.5, 127.3)
- added OL102: ~, SSL Footprints:main_board_outline_v3, F.Cu at (150.0, 92.0)
- added Q101: DMN21D2UFB-7B, SSL Footprints:DMN21D2UFB7B, F.Cu at (139.0, 57.0)
- added R102: 10k, Resistor_SMD:R_0402_1005Metric, F.Cu at (139.0, 59.0)
- added R106: 1k, Resistor_SMD:R_0402_1005Metric, F.Cu at (139.0, 58.0)
- added R107: 10k, Resistor_SMD:R_0402_1005Metric, F.Cu at (182.0, 100.5)
- added R127: 4k7, Resistor_SMD:R_0402_1005Metric, F.Cu at (181.0, 100.5)
- added R129: 10k, Resistor_SMD:R_0402_1005Metric, F.Cu at (154.5, 80.5)
- added R130: 10k, Resistor_SMD:R_0402_1005Metric, F.Cu at (159.2, 85.5)
- added R131: 10k, Resistor_SMD:R_0402_1005Metric, F.Cu at (158.2, 85.5)
- added R132: 10k, Resistor_SMD:R_0402_1005Metric, F.Cu at (169.2, 85.5)
- added R133: 10k, Resistor_SMD:R_0402_1005Metric, F.Cu at (170.2, 85.5)
- added R134: 10k, Resistor_SMD:R_0402_1005Metric, F.Cu at (158.2, 78.8)
- added R135: 6k8, Resistor_SMD:R_0402_1005Metric, F.Cu at (156.2, 78.8)
- added R136: 10k, Resistor_SMD:R_0402_1005Metric, F.Cu at (169.2, 78.8)
- added R137: 3k3, Resistor_SMD:R_0402_1005Metric, F.Cu at (167.2, 78.8)
- added R138: 10k, Resistor_SMD:R_0402_1005Metric, F.Cu at (165.5, 80.5)
- added U108: DRV8220DSGR, SSL Footprints:SON50P200X200X80-9N, F.Cu at (162.0, 123.0)
- added U109: TPS16416DRCR, SSL Footprints:TPS74901DRCR, F.Cu at (168.8, 81.8)
- added U110: TPS16416DRCR, SSL Footprints:TPS74901DRCR, F.Cu at (157.8, 81.8)
- C101, C102: footprint Capacitor_SMD:C_0603_1608Metric -> Capacitor_SMD:C_0402_1005Metric
- R105: value 10k -> 22k
- moved L103 139.4 mm to (146.0, 74.3), turned to -90 degrees
- moved L102 129.7 mm to (157.0, 74.2), turned to -90 degrees
- moved K101 126.7 mm to (124.9, 57.0)
- moved C129 126.5 mm to (148.2, 57.8), turned to 90 degrees
- moved R117 124.4 mm to (150.8, 68.5), turned to 90 degrees
- moved R119 121.8 mm to (158.2, 106.5), turned to 180 degrees
- moved R118 121.7 mm to (158.2, 104.0), turned to 180 degrees
- moved R116 121.7 mm to (150.8, 70.8), turned to 90 degrees
- moved C127 120.8 mm to (140.5, 75.5), turned to 90 degrees
- moved L101 120.6 mm to (168.0, 74.2), turned to -90 degrees
- moved C124 119.1 mm to (142.2, 75.5), turned to 90 degrees
- moved R111 118.8 mm to (158.2, 101.5), turned to 180 degrees
- moved U105 117.9 mm to (148.2, 67.8), turned to -90 degrees
- moved C128 115.8 mm to (159.2, 57.8), turned to 90 degrees
- moved C106 113.5 mm to (144.2, 67.8), turned to -90 degrees
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Connections:
- J109 pad 1: GND -> unconnected-(J109-Pin_1-Pad1)
- J109 pad 2: GND -> unconnected-(J109-Pin_2-Pad2)
- J109 pad 21: unconnected-(J109-Pin_21-Pad21) -> /MOTOR_PH
- J109 pad 23: unconnected-(J109-Pin_23-Pad23) -> /MOTOR_EN
- J109 pad 27: unconnected-(J109-Pin_27-Pad27) -> /ENC_A_3V3
- J109 pad 28: unconnected-(J109-Pin_28-Pad28) -> /~{SLEEP}
- J109 pad 29: unconnected-(J109-Pin_29-Pad29) -> /ENC_B_3V3
- J109 pad 30: unconnected-(J109-Pin_30-Pad30) -> /TRIG
- J109 pad 7: GND -> +3.3V
- K101 pad 11: unconnected-(K101-Pad11) -> /CAP
- K101 pad 12: unconnected-(K101-Pad12) -> /HV
- K101 pad 14: unconnected-(K101-Pad14) -> /COIL
- K101 pad A1: unconnected-(K101-PadA1) -> +5V
- K101 pad A2: unconnected-(K101-PadA2) -> /TRIG_D
- R125 pad 1: /3V3_UNFUSED -> /ENC_A_3V3
- R125 pad 2: /3V3_OVLO -> GND
- R126 pad 1: /3V3_OVLO -> /ENC_A
- R126 pad 2: GND -> /ENC_A_3V3
- U103 pad 2: unconnected-(U103-PGOOD-Pad2) -> /PGOOD_5V
- U104 pad 2: unconnected-(U104-PGOOD-Pad2) -> /PGOOD_3V3
Routing:
- net +5V: track 50.2 -> 197.0 mm, vias 2 -> 1
- net /TRIG: track 0.00 -> 96.9 mm, vias 0 -> 1
- net /Microcontroller/BTN2: track 92.2 -> 0.00 mm, vias 4 -> 0
- net GND: track 124.0 -> 36.2 mm, vias 449 -> 377
- net /Microcontroller/BTN1: track 82.3 -> 0.00 mm, vias 2 -> 0
- net /Microcontroller/TRIG1: track 77.3 -> 0.00 mm, vias 2 -> 0
- net /Microcontroller/TRIG2: track 60.8 -> 0.00 mm, vias 2 -> 0
- net /Microcontroller/NRST: track 56.3 -> 0.00 mm, vias 5 -> 0
- net /Microcontroller/CAN1_L: track 49.8 -> 0.00 mm
- net /HV: track 0.00 -> 41.7 mm
- net /Microcontroller/CAN1_H: track 40.6 -> 0.00 mm
- net /ENC_A: track 0.00 -> 38.9 mm, vias 0 -> 1
- net /ENC_B: track 0.00 -> 38.9 mm, vias 0 -> 1
- net /~{SLEEP}: track 0.00 -> 38.8 mm, vias 0 -> 1
- net +3.3V: track 92.1 -> 54.0 mm, vias 43 -> 1
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- added copper zone on F.Cu, net /3V3_UNFUSED
- added copper zone on F.Cu, net /5V_UNFUSED
- added copper zone on B.Cu, net /CAP
- added copper zone on F.Cu, net /CAP
- added copper zone on In1.Cu, net /CAP
- added copper zone on In2.Cu, net /CAP
- added copper zone on B.Cu, net /COIL
- added copper zone on F.Cu, net /COIL
- added copper zone on In1.Cu, net /COIL
- added copper zone on In2.Cu, net /COIL
- added copper zone on F.Cu, net /OUT1
- added copper zone on F.Cu, net /OUT2
- added copper zone on F.Cu, net /SW_12V
- added copper zone on F.Cu, net /SW_3V3
- added copper zone on F.Cu, net /SW_5V
- added copper zone on In2.Cu, net GND
- added copper zone on B.Cu, net GNDPWR
- added copper zone on F.Cu, net GNDPWR
- added copper zone on In1.Cu, net GNDPWR
- added copper zone on In2.Cu, net GNDPWR
- added copper zone on B.Cu, net VBAT
- removed copper zone on In2.Cu, net +3.3V
- removed copper zone on F.Cu, net /Power/SW_12V
- removed copper zone on F.Cu, net /Power/SW_3V3
- removed copper zone on F.Cu, net /Power/SW_5V
- removed copper zone on F.Cu, net /Power/TRIG1_D
- removed copper zone on F.Cu, net /Power/TRIG2_D
- removed copper zone on F.Cu, net VBUS
- removed copper zone on In2.Cu, net VSYS
Other:
- board size 100 x 95.5 mm -> 100 x 90.5 mm
- board text added: "BATTERY FAULT"
- board text added: "_{IMPERIAL SSL} Power Board v2.0"
- board text added: "max current on 3V3, 5V & 12V rails: 2A"
- board text removed: "+"
- board text removed: "-"
- board text removed: "Antenna switch 0: SMA 1: PCB"
- board text removed: "BAT IN"
- board text removed: "BAT OUT"
- board text removed: "BOOT"
- board text removed: "BTN1"
- board text removed: "BTN2"
- board text removed: "CAN1"
- board text removed: "CAN2"
- board text removed: "DEBUG"
- board text removed: "ERR"
- board text removed: "Max current on 3V3, 5V & 12V rails: 2A"
- board text removed: "RST"
- board text removed: "RUN"
- board text removed: "STAT"
- board text removed: "TRIG1"
- board text removed: "TRIG2"
- board text removed: "_{IMPERIAL SSL} Main Board v1.0"

Commit message: PCBs Done
Parts:
- moved G*** 9.24 mm to (146.0, 67.4)
- moved D106 3.85 mm to (143.4, 86.9)
Routing:
- net /CAP: track 34.9 -> 33.2 mm
Other:
- board text added: "Battery voltage: 12-25V"
- board text added: "CAP"
- board text added: "COIL"
- board text added: "HV"
- board text added: "MOTOR"
- board text added: "Max current on 3V3, 5V & 12V rails: 1A"
- board text added: "VBAT"
- board text added: "_{IMPERIAL SSL} Power Board v1.0"
- board text removed: "Battery voltage: 12-30V"
- board text removed: "_{IMPERIAL SSL} Power Board v2.0"
- board text removed: "max current on 3V3, 5V & 12V rails: 2A"
